File: Marshall 18 Watt/Marshall 18 Watt.kicad_pcb (KiCad board)
At the start: 2 copper layers, 37 parts, among them J1 LOW, J2 HIGH, J3 Conn_01x03_Socket, J4 Heater, U1 ECC83, U2 ECC83, U3 EL84, U4 EL84

Commit message: Update_17_03_25
Add sch
Parts:
- removed C16, C17: 0.01uF, Capacitor_THT:C_Axial_L5.1mm_D3.1mm_P10.00mm_Horizontal
- removed J2: HIGH, Connector_Audio:Jack_6.35mm_Neutrik_NMJ4HCD2_Horizontal
- removed R17: 47K, Resistor_THT:R_Axial_DIN0411_L9.9mm_D3.6mm_P20.32mm_Horizontal
- removed R18, R19: 100K, Resistor_THT:R_Axial_DIN0411_L9.9mm_D3.6mm_P20.32mm_Horizontal
- removed R20: 125/5W, Resistor_THT:R_Axial_DIN0411_L9.9mm_D3.6mm_P20.32mm_Horizontal
- removed R21, R22: 8.2K, Resistor_THT:R_Axial_DIN0411_L9.9mm_D3.6mm_P20.32mm_Horizontal
- removed R23: 470K, Resistor_THT:R_Axial_DIN0411_L9.9mm_D3.6mm_P20.32mm_Horizontal
- removed Tone1, Volume1: 500KA, Potentiometer_THT:Potentiometer_Alps_RK163_Single_Horizontal
- removed U4: EL84, Valve:Valve_Noval_P
- added Bass1: 250KA, Potentiometer_THT:Potentiometer_Alps_RK163_Single_Horizontal, F.Cu at (164.2, 129.5)
- added C10: 50-500uF/25V, Capacitor_THT:CP_Radial_D18.0mm_P7.50mm, F.Cu at (234.7, 44.1)
- added C12: 50-500uF/25V, Capacitor_THT:CP_Radial_D18.0mm_P7.50mm, F.Cu at (188.0, 43.6)
- added C13: 50-500uF/25V, Capacitor_THT:CP_Radial_D10.0mm_P3.80mm, F.Cu at (207.3, 22.5)
- added C2: 50uF/25V, Capacitor_THT:CP_Radial_D10.0mm_P3.80mm, F.Cu at (28.7, 91.4)
- added C4: 150pF, Capacitor_THT:C_Rect_L29.0mm_W7.6mm_P27.50mm_MKT, F.Cu at (114.3, 106.7)
- added C7: 47nF, Capacitor_THT:C_Rect_L29.0mm_W7.6mm_P27.50mm_MKT, F.Cu at (141.8, 97.5)
- added C8: 0.01uF, Capacitor_THT:C_Rect_L29.0mm_W7.6mm_P27.50mm_MKT, F.Cu at (152.4, 97.0)
- added C9: 50-500uF/25V, Capacitor_THT:CP_Radial_D10.0mm_P3.80mm, F.Cu at (194.3, 98.6)
- added D1: B40R, Diode_THT:Diode_Bridge_Round_D9.0mm, F.Cu at (242.9, 22.9)
- added D2: BZV55C6V2, Diode_THT:D_DO-15_P10.16mm_Horizontal, F.Cu at (196.1, 22.4)
- added Gain1: 250KA, Potentiometer_THT:Potentiometer_Alps_RK163_Single_Horizontal, F.Cu at (84.9, 129.5)
- added Gain2: 250KA, Potentiometer_THT:Potentiometer_Alps_RK163_Single_Horizontal, F.Cu at (124.5, 129.5)
- added Mid1: 25KA, Potentiometer_THT:Potentiometer_Alps_RK163_Single_Horizontal, F.Cu at (203.8, 129.6)
- added R11: 100K/2W, Resistor_THT:R_Axial_DIN0411_L9.9mm_D3.6mm_P20.32mm_Horizontal, F.Cu at (189.5, 51.8)
- added R12: 100K/2W, Resistor_THT:R_Axial_DIN0411_L9.9mm_D3.6mm_P20.32mm_Horizontal, F.Cu at (234.7, 51.8)
- added R14: 125/5W, Resistor_THT:R_Axial_DIN0411_L9.9mm_D3.6mm_P20.32mm_Horizontal, F.Cu at (232.7, 101.7)
- added Treble1: 250KA, Potentiometer_THT:Potentiometer_Alps_RK163_Single_Horizontal, F.Cu at (243.4, 129.5)
- C1: footprint Capacitor_THT:C_Axial_L5.1mm_D3.1mm_P10.00mm_Horizontal -> Capacitor_THT:C_Rect_L29.0mm_W7.6mm_P27.50mm_MKT
- C11: value 50uF/25V -> 50-500uF/25V; footprint Capacitor_THT:CP_Radial_D8.0mm_P5.00mm -> Capacitor_THT:CP_Radial_D18.0mm_P7.50mm
- C3: value 50-500uF/25V -> 0.01uF; footprint Capacitor_THT:CP_Radial_D8.0mm_P5.00mm -> Capacitor_THT:C_Rect_L29.0mm_W7.6mm_P27.50mm_MKT
- C5: value 0.05uF -> 22nF; footprint Capacitor_THT:C_Axial_L5.1mm_D3.1mm_P10.00mm_Horizontal -> Capacitor_THT:C_Rect_L29.0mm_W7.6mm_P27.50mm_MKT
- C6: value 0.01uF -> 22nF; footprint Capacitor_THT:C_Axial_L5.1mm_D3.1mm_P10.00mm_Horizontal -> Capacitor_THT:C_Rect_L29.0mm_W7.6mm_P27.50mm_MKT
- J1: value LOW -> Conn_01x02_Socket; footprint Connector_Audio:Jack_6.35mm_Neutrik_NMJ4HCD2_Horizontal -> Connector_PinSocket_2.54mm:PinSocket_1x02_P2.54mm_Vertical
- J3: footprint Connector_Phoenix_MC_HighVoltage:PhoenixContact_MCV_1,5_3-G-5.08_1x03_P5.08mm_Vertical -> Connector_Phoenix_MC_HighVoltage:PhoenixContact_MCV_1,5_3-GF-5.08_1x03_P5.08mm_Vertical_ThreadedFlange
- J4: value Heater -> NMJ4HHD2; footprint Connector_Phoenix_MC_HighVoltage:PhoenixContact_MCV_1,5_2-G-5.08_1x02_P5.08mm_Vertical -> Connector_Audio:Jack_6.35mm_Neutrik_NMJ4HHD2_Horizontal
- R1: value R -> 1M
- R10: value 81.5K-2K/2W -> 100K
- R13: value 820 -> 8.2K
- R15: value 470K -> 680/3W
- R16: value 470K -> 100K/2W
- R2: value 820 -> 68K
- R3: value 1M -> 1K5
- R4: value 1M -> 100K
- R5, R7: value 100K -> 1M
- R6: value 8.2K/2W -> 68K
- R8: value 100/3W -> 820
- R9: value 470K -> 39K
- U1: value ECC83 -> 12AX7; footprint Valve:Valve_Noval_P -> Elab:9P_2.57mm
- U2: value ECC83 -> EZ80; footprint Valve:Valve_Noval_P -> Elab:9P_2.57mm
- U3: footprint Valve:Valve_Noval_P -> Elab:9P_2.57mm
- moved J1 212.1 mm to (257.0, 26.6)
- moved J3 177.3 mm to (257.6, 68.6), turned to 90 degrees
- moved R16 159.0 mm to (235.7, 22.9), turned to 180 degrees
- moved C11 152.6 mm to (211.8, 44.1), turned to 90 degrees
- moved U2 126.7 mm to (193.5, 84.3)
- moved R9 126.5 mm to (80.8, 112.8)
- moved C6 124.6 mm to (179.4, 107.2)
- moved J4 116.7 mm to (40.6, 116.8), turned to -90 degrees
- moved C5 110.0 mm to (152.4, 116.3)
- moved R15 109.5 mm to (232.7, 106.7)
- moved R7 106.2 mm to (101.1, 106.7), turned to 180 degrees
- moved C3 104.3 mm to (47.7, 107.7)
- moved R1 98.4 mm to (71.6, 119.9), turned to 180 degrees
- moved R3 71.0 mm to (20.3, 101.1)
- moved R2 62.5 mm to (71.6, 114.3), turned to 180 degrees
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Connections:
- C1 pad 2: Net-(U2B-G) -> Net-(C1-Pad2)
- C11 pad 1: Net-(U1A-K) -> Net-(U3A-A)
- C11 pad 2: GNDPWR -> GND
- C3 pad 1: Net-(U3A-K_G3) -> Net-(U1A-A)
- C3 pad 2: GNDPWR -> Net-(C3-Pad2)
- C5 pad 1: Net-(U1A-A) -> Net-(C5-Pad1)
- C5 pad 2: Net-(C5-Pad2) -> Net-(Bass1-Pad1)
- C6 pad 1: Net-(U1A-A) -> Net-(C5-Pad1)
- J3 pad 3: Net-(J3-Pin_3) -> GND
- R1 pad 1: unconnected-(R1-Pad1) -> Net-(C1-Pad2)
- R1 pad 2: unconnected-(R1-Pad2) -> GND
- R10 pad 1: Net-(R10-Pad1) -> Net-(C12-Pad1)
- R10 pad 2: Net-(J3-Pin_2) -> Net-(U1B-A)
- R13 pad 1: Net-(U2A-K) -> Net-(Gain2-Pad2)
- R13 pad 2: Net-(R13-Pad2) -> Net-(U3A-G1)
- R15 pad 1: Net-(C16-Pad2) -> Net-(U3A-G2)
- R15 pad 2: GNDPWR -> Net-(U3A-A)
- R16 pad 2: GNDPWR -> Net-(D2-K)
- R2 pad 1: Net-(U1A-K) -> Net-(C1-Pad2)
- R2 pad 2: GNDPWR -> Net-(U1A-G)
- R3 pad 1: Net-(U1B-G) -> Net-(U1A-K)
- R3 pad 2: GNDPWR -> GND
- R4 pad 1: Net-(U1A-G) -> Net-(C12-Pad1)
- R4 pad 2: GNDPWR -> Net-(U1A-A)
- R5 pad 1: Net-(C5-Pad2) -> Net-(C3-Pad2)
- R5 pad 2: Net-(R5-Pad2) -> GND
- R6 pad 1: Net-(R18-Pad1) -> Net-(C4-Pad1)
- R6 pad 2: Net-(R10-Pad1) -> Net-(C5-Pad1)
- R7 pad 1: Net-(R18-Pad1) -> Net-(U1B-G)
- R7 pad 2: Net-(U1A-A) -> Net-(R7-Pad2)
- R8 pad 1: Net-(U3A-G2) -> Net-(U1B-K)
- R8 pad 2: Net-(R10-Pad1) -> Net-(R7-Pad2)
- R9 pad 1: Net-(U2B-G) -> Net-(R7-Pad2)
- R9 pad 2: Net-(R13-Pad2) -> GND
- U1 pad 1: Net-(U1A-A) -> Net-(U1B-A)
- U1 pad 3: Net-(U1A-K) -> Net-(U1B-K)
- U1 pad 4: Net-(J4-Pin_1) -> Net-(D2-K)
- U1 pad 5: Net-(J4-Pin_1) -> Net-(D2-K)
- U1 pad 9: Net-(J4-Pin_2) -> Net-(D1--)
- U2 pad 1: Net-(U2B-A) -> Net-(J3-Pin_2)
- U2 pad 2: Net-(U2B-G) -> (no net)
- U2 pad 4: Net-(J4-Pin_1) -> Net-(D2-K)
- U2 pad 5: Net-(J4-Pin_1) -> Net-(D1--)
- U2 pad 6: Net-(U2A-A) -> (no net)
- U2 pad 7: Net-(U2A-G) -> Net-(J3-Pin_1)
- U2 pad 8: Net-(U2A-K) -> (no net)
- U2 pad 9: Net-(J4-Pin_2) -> (no net)
- U3 pad 4: Net-(J4-Pin_1) -> Net-(D2-K)
- U3 pad 5: Net-(J4-Pin_2) -> Net-(D1--)
- U3 pad 7: Net-(J3-Pin_1) -> Net-(U3A-A)
Routing:
- net Net-(U1B-A): track 0.00 -> 83.9 mm
- net Net-(U1B-K): track 0.00 -> 43.0 mm
- net Net-(U1A-A): track 0.00 -> 40.1 mm
- net Net-(U1B-G): track 52.4 -> 80.1 mm
- net Net-(C3-Pad2): track 0.00 -> 27.1 mm
- net Net-(U1A-G): track 75.1 -> 49.3 mm
- net Net-(U1A-K): track 28.1 -> 49.3 mm
- net Net-(C1-Pad2): track 0.00 -> 15.9 mm
- net Net-(C1-Pad1): track 0.00 -> 8.64 mm
- net Net-(R7-Pad2): track 0.00 -> 6.10 mm
- net Net-(J4-Pin_1): track 5.08 -> 0.00 mm
- added copper zone on B.Cu, net GND

Commit message: Update 18_03_25
V01
Parts:
- removed C13: 50-500uF/25V, Capacitor_THT:CP_Radial_D10.0mm_P3.80mm
- removed D1: B40R, Diode_THT:Diode_Bridge_Round_D9.0mm
- removed D2: BZV55C6V2, Diode_THT:D_DO-15_P10.16mm_Horizontal
- removed R16: 100K/2W, Resistor_THT:R_Axial_DIN0411_L9.9mm_D3.6mm_P20.32mm_Horizontal
- added H1: GND, MountingHole:MountingHole_2.7mm_Pad_Via, F.Cu at (22.9, 68.0)
- added H2: GND, MountingHole:MountingHole_2.7mm_Pad_Via, F.Cu at (59.7, 130.8)
- added H3: GND, MountingHole:MountingHole_2.7mm_Pad_Via, F.Cu at (269.2, 132.1)
- added H4: GND, MountingHole:MountingHole_2.7mm_Pad_Via, F.Cu at (269.2, 67.3)
- added J2: Heater, Connector_Phoenix_MC_HighVoltage:PhoenixContact_MCV_1,5_2-G-5.08_1x02_P5.08mm_Vertical, F.Cu at (249.2, 83.3)
- J1: footprint Connector_PinSocket_2.54mm:PinSocket_1x02_P2.54mm_Vertical -> Connector_Audio:Jack_6.35mm_Neutrik_NMJ4HCD2_Horizontal
- J3: value Conn_01x03_Socket -> Conn_01x03_Pin; footprint Connector_Phoenix_MC_HighVoltage:PhoenixContact_MCV_1,5_3-GF-5.08_1x03_P5.08mm_Vertical_ThreadedFlange -> Connector_Phoenix_MC_HighVoltage:PhoenixContact_MCV_1,5_3-G-5.08_1x03_P5.08mm_Vertical
- J4: value NMJ4HHD2 -> OT; footprint Connector_Audio:Jack_6.35mm_Neutrik_NMJ4HHD2_Horizontal -> Connector_Phoenix_MC_HighVoltage:PhoenixContact_MCV_1,5_3-G-5.08_1x03_P5.08mm_Vertical
- moved J1 234.4 mm to (40.6, 116.8), turned to -90 degrees
- moved R14 131.8 mm to (101.2, 92.7)
- moved J4 115.9 mm to (151.7, 83.5), turned to 0 degrees
- moved R15 97.3 mm to (136.4, 92.7)
- moved R13 92.4 mm to (141.0, 111.3), turned to 180 degrees
- moved C9 90.8 mm to (104.8, 83.4), turned to 180 degrees
- moved C4 75.6 mm to (189.7, 101.6), turned to -90 degrees
- moved C12 65.7 mm to (216.0, 103.0), turned to -90 degrees
- moved C11 63.6 mm to (235.6, 103.1), turned to -90 degrees
- moved C10 62.6 mm to (255.1, 103.3), turned to -90 degrees
- moved R12 53.4 mm to (203.5, 95.1), turned to -90 degrees
- moved C7 45.6 mm to (108.7, 128.9), turned to 90 degrees
- moved R11 44.0 mm to (197.2, 95.1), turned to -90 degrees
- moved J3 37.4 mm to (223.2, 83.3), turned to 0 degrees
- moved C8 36.8 mm to (116.2, 103.6)
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Connections:
- C10 pad 1: Net-(U2A-K) -> B+
- C11 pad 1: Net-(U3A-A) -> B2+
- C2 pad 1: Net-(U1A-K) -> Net-(U1B-K)
- C3 pad 1: Net-(U1A-A) -> Net-(U1B-A)
- C4 pad 1: Net-(C4-Pad1) -> Net-(C3-Pad2)
- C7 pad 2: Net-(U1B-G) -> Net-(U1A-G)
- C8 pad 1: Net-(U1B-A) -> Net-(U1A-A)
- Gain1 pad 1: Net-(C3-Pad2) -> Net-(Gain1-Pad1)
- Gain1 pad 2: Net-(C4-Pad1) -> Net-(C7-Pad1)
- R10 pad 2: Net-(U1B-A) -> Net-(U1A-A)
- R11 pad 2: Net-(U3A-A) -> B2+
- R12 pad 1: Net-(U2A-K) -> B+
- R12 pad 2: Net-(U3A-A) -> B2+
- R15 pad 2: Net-(U3A-A) -> Net-(J4-Pin_2)
- R2 pad 2: Net-(U1A-G) -> Net-(U1B-G)
- R3 pad 1: Net-(U1A-K) -> Net-(U1B-K)
- R4 pad 2: Net-(U1A-A) -> Net-(U1B-A)
- R6 pad 1: Net-(C4-Pad1) -> Net-(C3-Pad2)
- R7 pad 1: Net-(U1B-G) -> Net-(U1A-G)
- R8 pad 1: Net-(U1B-K) -> Net-(U1A-K)
- Treble1 pad 2: Net-(C7-Pad1) -> Net-(Gain1-Pad1)
- U2 pad 3: Net-(U2A-K) -> B+
- U3 pad 7: Net-(U3A-A) -> Net-(J4-Pin_2)
Routing:
- net Net-(J2-Pin_2): track 0.00 -> 272.6 mm, vias 0 -> 4
- net Net-(Gain1-Pad1): track 0.00 -> 221.2 mm
- net Net-(J2-Pin_1): track 0.00 -> 211.3 mm, vias 0 -> 4
- net Net-(C12-Pad1): track 0.00 -> 156.9 mm, vias 0 -> 2
- net Net-(Bass1-Pad1): track 0.00 -> 122.2 mm
- net B+: track 0.00 -> 111.8 mm
- net Net-(C3-Pad2): track 27.1 -> 137.6 mm
- net Net-(U1B-G): track 80.1 -> 19.1 mm
- net Net-(J4-Pin_2): track 0.00 -> 57.2 mm
- net Net-(C4-Pad2): track 0.00 -> 56.5 mm
- net Net-(U1B-A): track 83.9 -> 28.1 mm
- net Net-(U1A-A): track 40.1 -> 95.3 mm
- net Net-(Bass1-Pad3): track 0.00 -> 52.7 mm
- net B2+: track 0.00 -> 46.4 mm
- net Net-(J3-Pin_1): track 0.00 -> 43.0 mm
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- added copper zone on F.Cu, net GND
Other:
- board outline added: 255.5 x 73.4 mm
