File: Marshall 18 Watt/Marshall 18 Watt.kicad_sch (KiCad schematic)
At the start: 36 parts, among them J1 LOW, J2 Heater, U1 ECC83, U2 EZ80, U3 EL84

Commit message: Update 18_03_25
V01
Parts:
- added C12: 50-500uF/25V, Capacitor_THT:CP_Radial_D18.0mm_P7.50mm, symbol Device:C_Polarized_US
- added H1, H2, H3, H4: GND, MountingHole:MountingHole_2.5mm_Pad_TopBottom, symbol Mechanical:MountingHole_Pad
- added J3: Conn_01x03_Pin, Connector_Phoenix_MC_HighVoltage:PhoenixContact_MCV_1,5_3-G-5.08_1x03_P5.08mm_Vertical, symbol Connector:Conn_01x03_Pin
- added J4: OT, Connector_Phoenix_MC_HighVoltage:PhoenixContact_MCV_1,5_3-G-5.08_1x03_P5.08mm_Vertical, symbol Connector:Conn_01x03_Pin
- C1, C4, C5, C6, C7, C8: footprint Capacitor_THT:C_Axial_L5.1mm_D3.1mm_P10.00mm_Horizontal -> Capacitor_THT:C_Rect_L29.0mm_W7.6mm_P27.50mm_MKT
- C10, C11: footprint Capacitor_THT:CP_Radial_D8.0mm_P5.00mm -> Capacitor_THT:CP_Radial_D18.0mm_P7.50mm
- C2, C9: footprint Capacitor_THT:CP_Radial_D8.0mm_P5.00mm -> Capacitor_THT:CP_Radial_D10.0mm_P3.80mm
- C3: footprint Capacitor_THT:CP_Radial_D8.0mm_P5.00mm -> Capacitor_THT:C_Rect_L29.0mm_W7.6mm_P27.50mm_MKT
- J1: value LOW -> Conn_01x02_Socket
- J2: footprint Connector_Audio:Jack_6.35mm_Neutrik_NMJ4HCD2_Horizontal -> Connector_Phoenix_MC_HighVoltage:PhoenixContact_MCV_1,5_2-G-5.08_1x02_P5.08mm_Vertical
- R11: value 8.2K/2W -> 100K/2W
- U1: value ECC83 -> 12AX7; footprint Valve:Valve_Noval_P -> Elab:9P_2.57mm
- U2, U3: footprint Valve:Valve_Noval_P -> Elab:9P_2.57mm
Connections:
- net GND: now also J1.TN, C12.2, H1.1, H2.1, H3.1, H4.1, J3.3 (Pin_3), J4.1 (Pin_1)
- net at C7.1: now also Gain1.2; no longer Treble1.2
- net at U1.4 (F1), U1.5 (F1), U2.4 (H)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: now also J2.2 (Pin_2); no longer J2.1 (Pin_1)
- net at U1.9 (F2), U2.5 (H), U3.5 (F2): now also J2.1 (Pin_1); no longer J2.2 (Pin_2)
- net B+: now reaches C10.1, R12.1, U2.3 (K)
- net B+: now also J4.3 (Pin_3)
- net at R10.1, R11.1, R4.1: now also C12.1
- net B2+: now reaches C11.1, R12.2
- net B2+: now also R11.2
- net at R15.2, U3.7 (A): now also J4.2 (Pin_2); no longer R11.2
- net at U2.1 (A): now also J3.2 (Pin_2)
- net at U2.7 (A): now also J3.1 (Pin_1)
- net at C3.2, R5.1: now also C4.1, R6.1; no longer Gain1.1
- new net: Gain1.1, Treble1.2
Other:
- moved on the sheet: Bass1, C11, C4, C5, C6, C7, Gain1, Mid1, R11, R12, R6, Treble1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
