File: Marshall 18 Watt/PT2399_Delay/PT2399_Delay.kicad_sch (KiCad schematic)
At the start: 52 parts, among them J1 +9V, J2 IN, J3 IN, U1 PT2399, U2 TL072, U3 L7805

Commit message: update_26_03_25
Rev Delay
Parts:
- U2: footprint (none) -> Package_DIP:DIP-8_W7.62mm
- renumbered C20 to C1, C16 to C10, C10 to C11, C11 to C12, C8 to C13, C1 to C14, C18 to C16, C13 to C17, C12 to C18, C6 to C19, C21 to C2, C17 to C20, C19 to C21, C7 to C22, C22 to C3, C2 to C5, C3 to C6, C5 to C7, C9 to C8, C14 to C9, FDBK to FDBK2, J2 to J1, J1 to J2, MIX to MIX1, R13 to R10, R14 to R11, R17 to R12, R15 to R13, R12 to R14, R7 to R15, R8 to R17, R4 to R2, R9 to R20, R20 to R3, R2 to R4, R3 to R5, R5 to R6, R6 to R7, R11 to R8, R10 to R9

Commit message: Update _26_03_25
PCB
Parts:
- removed J2: +9V, Connector_BarrelJack:BarrelJack_GCT_DCJ200-10-A_Horizontal, symbol Connector:Barrel_Jack_MountingPin
- added D2: IR204A, LED_THT:LED_D3.0mm_IRBlack, symbol LED:IR204A
- added J2: Barrel_Jack_Switch, Connector_BarrelJack:BarrelJack_GCT_DCJ200-10-A_Horizontal, symbol Connector:Barrel_Jack_Switch
- added J4: IN, Connector_JST:JST_XA_B02B-XASK-1_1x02_P2.50mm_Vertical, symbol Connector:Conn_01x02_Pin
- added R21: 10k, Resistor_THT:R_Axial_DIN0204_L3.6mm_D1.6mm_P5.08mm_Horizontal, symbol Device:R
- C14, C5, C6: footprint Capacitor_THT:CP_Radial_D4.0mm_P2.00mm -> Capacitor_THT:CP_Radial_D5.0mm_P2.50mm
- FDBK1, FDBK2, MIX1: footprint Potentiometer_THT:Potentiometer_Alps_RK163_Single_Horizontal -> Potentiometer_THT:Potentiometer_Omeg_PC16BU_Vertical
Connections:
- net GND: now also J2.2, J2.3, J4.2 (Pin_2), R21.1
- net GNDA: now also J4.1 (Pin_1)
- net VDD: now also U1.1 (VCC), D2.2 (A)
- net at R1.1: now also J2.1
- new net: D2.1 (K), R21.2
