File: TubeScreamer/TS/TS.kicad_sch (KiCad schematic)
At the start: 80 parts, among them J1 DC 9V, J2 BAT, J3 IN, J4 OUT, Q1 2SC1815, Q2 2SK44SP, Q3 2SC1815, Q4 2SC1815, Q5 2SC1815, Q6 2SC1815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

Commit message: Update 27_03_15
sch TS fix
Parts:
- RV1, RV2, RV3: footprint Potentiometer_THT:Potentiometer_Omeg_PC16BU_Vertical -> Connector_PinHeader_2.54mm:PinHeader_1x03_P2.54mm_Vertical
Changed lines of the file:
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@@
       (effects (font (size 1.27 1.27)) (justify right))
     )
-    (property "Footprint" "Potentiometer_THT:Potentiometer_Omeg_PC16BU_Vertical" (at 186.69 81.28 0)
+    (property "Footprint" "Connector_PinHeader_2.54mm:PinHeader_1x03_P2.54mm_Vertical" (at 186.69 81.28 0)
       (effects (font (size 1.27 1.27)) hide)
     )
@@
       (effects (font (size 1.27 1.27)))
     )
-    (property "Footprint" "Potentiometer_THT:Potentiometer_Omeg_PC16BU_Vertical" (at 114.3 38.1 0)
+    (property "Footprint" "Connector_PinHeader_2.54mm:PinHeader_1x03_P2.54mm_Vertical" (at 114.3 38.1 0)
       (effects (font (size 1.27 1.27)) hide)
     )
@@
       (effects (font (size 1.27 1.27)))
     )
-    (property "Footprint" "Potentiometer_THT:Potentiometer_Omeg_PC16BU_Vertical" (at 140.97 57.15 0)
-      (effects (font (size 1.27 1.27)) hide)
-    )
+    (property "Footprint" "Connector_PinHeader_2.54mm:PinHeader_1x03_P2.54mm_Vertical" (at 140.97 57.15 0)
+      (effects (font (size 1.27 1.27)) hide)
+    )
